File: sdt_pa_diode.kicad_sch (KiCad schematic)
At the start: 10 parts

Commit message: First layout started.
Parts:
- removed U?: TMP36GRTZ-REEL7, SOT95P280X145-5N, symbol TMP36GRTZ-REEL7:TMP36GRTZ-REEL7
- added C1, C2, C3, C4: C_Small, Capacitor_SMD:C_1206_3216Metric_Pad1.33x1.80mm_HandSolder, symbol Device:C_Small
- added J1: Conn_01x05, Connector_PinHeader_2.54mm:PinHeader_1x05_P2.54mm_Horizontal, symbol Connector_Generic:Conn_01x05
- added R1: R_US, Resistor_SMD:R_1206_3216Metric_Pad1.30x1.75mm_HandSolder, symbol Device:R_US
- added U1: TMP36GRTZ-REEL7, TMP36GRTZ:TMP36GRTZ-REEL7, symbol TMP36GRTZ:TMP36GRTZ-REEL7
- gave numbers to parts that had none: 9
Connections:
- net GND: now also C1.2, C2.1, C3.2, C4.2, J1.2 (Pin_2), U1.3 (NC), U1.5 (GND)
- net at D1.2 (A): now also C2.2, J1.1 (Pin_1)
- new net +VS: C3.1, J1.4 (Pin_4), R1.2, U1.2 (+VS)
- new net SHUTDOWN*: C4.1, J1.3 (Pin_3), R1.1, U1.4 (SHUTDOWN*)
- new net VOUT: C1.1, J1.5 (Pin_5), U1.1 (VOUT)
Other:
- company: (none) -> SDT Not Incorporated
- title: (none) -> Power Amplifer Diode Sensor
- moved on the sheet: D1, D2, D3, D4, D5, D6, D7, D8, D9
