File: sdt_pa_diode.kicad_pcb (KiCad board)
At the start: 2 copper layers, 35 x 20 mm, 16 parts, among them J1 Conn_01x05, U1 TMP36GRTZ-REEL7

Commit message: Ready for first fab.
Parts:
- C1, C2, C3, C4, R1: moved to B.Cu
- U1: value TMP36GRTZ-REEL7 -> RJ_5_ADI; moved to B.Cu
- moved U1 22.6 mm to (145.6, 95.1)
- moved C1 21.5 mm to (148.4, 101.0), turned to 180 degrees
- moved R1 17.2 mm to (149.9, 96.2), turned to -90 degrees
- moved C2 16.0 mm to (148.7, 87.6), turned to 0 degrees
- moved C3 15.4 mm to (144.1, 89.5), turned to 90 degrees
- moved C4 14.1 mm to (148.7, 90.8), turned to 180 degrees
- moved J1 12.1 mm to (153.5, 89.8)
- moved D1 4.16 mm to (145.3, 87.4)
- moved D2 3.25 mm to (139.2, 87.4)
- moved D9 2.63 mm to (145.3, 102.5)
- moved D8 1.91 mm to (139.2, 102.5)
- moved D6 1.81 mm to (126.6, 102.5)
- moved D3 1.59 mm to (132.8, 87.4)
- moved D7 1.59 mm to (132.9, 102.5)
- moved D5 1.08 mm to (125.0, 95.0)
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Routing:
- net /+VS: track 0.00 -> 16.2 mm
- net /VOUT: track 0.00 -> 12.5 mm
- net Net-(C2-Pad2): track 0.00 -> 11.6 mm
- net /SHUTDOWN*: track 0.00 -> 10.8 mm
- net Net-(D4-Pad1): track 0.00 -> 5.95 mm
- net Net-(D5-Pad1): track 0.00 -> 5.90 mm
- net Net-(D6-Pad1): track 0.00 -> 3.00 mm
- net Net-(D2-Pad1): track 0.00 -> 3.00 mm
- net Net-(D7-Pad1): track 0.00 -> 2.95 mm
- net Net-(D3-Pad1): track 0.00 -> 2.95 mm
- net Net-(D8-Pad1): track 0.00 -> 2.90 mm
- net Net-(D1-Pad1): track 0.00 -> 2.90 mm
- net GND: vias 0 -> 18
- added copper zone on B.Cu, net GND
- added copper zone on F.Cu, net GND
